Commit message: load obj workinf

File: models/Phone/103251/mobility.urdf (robot description, URDF)
Before this commit: robot partnet_2435be698167b2167120841458f79dbe, 24 links, 23 joints
Joints:
- joint joint_22: origin xyz=0 0 0 rpy=1.570796326794897 0 -1.570796326794897 -> xyz=0 0 0 rpy=3.1415926 3.1415926 -1.570796326794897

File: models/Phone/103813/mobility.urdf (robot description, URDF)
Before this commit: robot partnet_7bdffa69c49eb1d7bf653fdedcac4c5b-4, 9 links, 8 joints
Joints:
- joint joint_7: origin xyz=0 0 0 rpy=1.570796326794897 0 -1.570796326794897 -> xyz=0 0 0 rpy=3.1415926 3.1415926 -1.570796326794897

File: models/Phone/103828/mobility.urdf (robot description, URDF)
Before this commit: robot partnet_86f9108ac5df3150afeee5da21ab102b-0, 3 links, 2 joints
Joints:
- joint joint_1: origin xyz=0 0 0 rpy=1.570796326794897 0 -1.570796326794897 -> xyz=0 0 0 rpy=3.1415926 3.1415926 -1.570796326794897

File: models/Phone/103892/mobility.urdf (robot description, URDF)
Before this commit: robot partnet_b1feb3020d9380ba4fb324159a14f34e, 23 links, 22 joints
Joints:
- joint joint_21: origin xyz=0 0 0 rpy=1.570796326794897 0 -1.570796326794897 -> xyz=0 0 0 rpy=3.1415926 3.1415926 -1.570796326794897

File: models/Phone/103916/mobility.urdf (robot description, URDF)
Before this commit: robot partnet_c3abf1c29ad0c7223a60d90fdaaee16f-2, 6 links, 5 joints
Joints:
- joint joint_4: origin xyz=0 0 0 rpy=1.570796326794897 0 -1.570796326794897 -> xyz=0 0 0 rpy=3.1415926 3.1415926 -1.570796326794897

File: models/Phone/103927/mobility.urdf (robot description, URDF)
Before this commit: robot partnet_e156db6fe3b9286c87cb3c64e47598b4, 9 links, 8 joints
Joints:
- joint joint_7: origin xyz=0 0 0 rpy=1.570796326794897 0 -1.570796326794897 -> xyz=0 0 0 rpy=3.1415926 3.1415926 -1.570796326794897

File: models/Remote/100269/mobility.urdf (robot description, URDF)
Before this commit: robot partnet_200065ca496c39086372ead55db87fa8, 46 links, 45 joints
Joints:
- joint joint_44: origin xyz=0 0 0 rpy=1.570796326794897 0 -1.570796326794897 -> xyz=0 0 0 rpy=3.1415926 3.1415926 -1.570796326794897

File: models/Remote/100270/mobility.urdf (robot description, URDF)
Before this commit: robot partnet_2053bdd83749adcc1e5c09d9fe5c0c76, 48 links, 47 joints
Joints:
- joint joint_46: origin xyz=0 0 0 rpy=1.570796326794897 0 -1.570796326794897 -> xyz=0 0 0 rpy=3.1415926 3.1415926 -1.570796326794897

File: models/Remote/100392/mobility.urdf (robot description, URDF)
Before this commit: robot partnet_2c6493d31849c15a75f1efca97bee05a, 44 links, 43 joints
Joints:
- joint joint_42: origin xyz=0 0 0 rpy=1.570796326794897 0 -1.570796326794897 -> xyz=0 0 0 rpy=3.1415926 3.1415926 -1.570796326794897

File: models/Remote/100394/mobility.urdf (robot description, URDF)
Before this commit: robot partnet_28f2a5df4a926c3e140a527375fd6757, 35 links, 34 joints
Joints:
- joint joint_33: origin xyz=0 0 0 rpy=1.570796326794897 0 -1.570796326794897 -> xyz=0 0 0 rpy=3.1415926 3.1415926 -1.570796326794897

File: models/Remote/100809/mobility.urdf (robot description, URDF)
Before this commit: robot partnet_61c6c6a47e5b9d34496c7671bf276db5, 59 links, 58 joints
Joints:
- joint joint_57: origin xyz=0 0 0 rpy=1.570796326794897 0 -1.570796326794897 -> xyz=0 0 0 rpy=3.1415926 3.1415926 -1.570796326794897

File: models/Remote/100819/mobility.urdf (robot description, URDF)
Before this commit: robot partnet_67919afe61a6a5f06bba06dda7e10cee, 39 links, 38 joints
Joints:
- joint joint_37: origin xyz=0 0 0 rpy=1.570796326794897 0 -1.570796326794897 -> xyz=0 0 0 rpy=3.1415926 3.1415926 -1.570796326794897

File: models/Remote/100997/mobility.urdf (robot description, URDF)
Before this commit: robot partnet_7852a457e59fd546d26c2593d1870bdb, 44 links, 43 joints
Joints:
- joint joint_42: origin xyz=0 0 0 rpy=1.570796326794897 0 -1.570796326794897 -> xyz=0 0 0 rpy=3.1415926 3.1415926 -1.570796326794897

File: models/Remote/101034/mobility.urdf (robot description, URDF)
Before this commit: robot partnet_c2540a2e0b927f34453782ca938ffcf1, 14 links, 13 joints
Joints:
- joint joint_12: origin xyz=0 0 0 rpy=1.570796326794897 0 -1.570796326794897 -> xyz=0 0 0 rpy=3.1415926 3.1415926 -1.570796326794897
