Commit message: load containers

File: models/Box/100243/mobility.urdf (robot description, URDF)
Before this commit: robot partnet_c7a2224b009756cc226245d28c34a910, 3 links, 2 joints
Links:
- removed link link_0
Joints:
- removed joint joint_0

File: models/Box/100247/mobility.urdf (robot description, URDF)
Before this commit: robot partnet_d2200aed9cbb4cacb38d5f389c7b61db, 3 links, 2 joints
Links:
- removed link link_0
Joints:
- removed joint joint_0

File: models/Suitcase/100550/mobility.urdf (robot description, URDF)
Before this commit: robot partnet_5f3af8ff93de34c9e7922afdefd88b6e, 4 links, 3 joints
Joints:
- joint joint_0: limit lower=0.0 upper=1.5707963267948966 -> lower=0 upper=1.5707963267948966
- joint joint_2: origin xyz=0 0 0 rpy=1.570796326794897 0 -1.570796326794897 -> xyz=0 0 0 rpy=3.1415926 3.1415926 -1.570796326794897

File: models/Suitcase/101668/mobility.urdf (robot description, URDF)
Before this commit: robot partnet_547ad62bd93988fff0117851f0671fde, 6 links, 5 joints
Joints:
- joint joint_4: origin xyz=0 0 0 rpy=1.570796326794897 0 -1.570796326794897 -> xyz=0 0 0 rpy=3.1415926 3.1415926 -1.570796326794897

File: models/Suitcase/103755/mobility.urdf (robot description, URDF)
Before this commit: robot partnet_6eee2279c193892a8c80080da8fd52c9-0, 4 links, 3 joints
Joints:
- joint joint_2: origin xyz=0 0 0 rpy=1.570796326794897 0 -1.570796326794897 -> xyz=0 0 0 rpy=3.1415926 3.1415926 -1.570796326794897

File: models/Suitcase/103761/mobility.urdf (robot description, URDF)
Before this commit: robot partnet_c93fdcf6017f435c3dd5925057fea065-0, 4 links, 3 joints
Joints:
- joint joint_2: origin xyz=0 0 0 rpy=1.570796326794897 0 -1.570796326794897 -> xyz=0 0 0 rpy=3.1415926 3.1415926 -1.570796326794897
