Commit message: grasp real objects

File: models/Dispenser/101458/mobility.urdf (robot description, URDF)
Before this commit: robot partnet_2cb950b9-43d6-4d7d-8352-2f70c936dd6a, 6 links, 5 joints
Links:
- link link_2: mass None -> 0.2

File: models/Safe/101363/mobility.urdf (robot description, URDF)
Before this commit: robot partnet_019dff2f-8207-4ddf-8255-871060cd4bf6, 4 links, 3 joints
Links:
- removed link link_0
- removed link link_1
- link link_2: geometry collision mesh filename=textured_objs/original-3-back.obj; collision mesh filename=textured_objs/original-3-bottom.obj
Joints:
- removed joint joint_0
- removed joint joint_1
