Commit message: pack mug & stapler

File: models/Mug/7008/mobility.urdf (robot description, URDF)
Before this commit: robot Mug_159e56c18906830278d8f8c02c47cde0_M, 2 links, 1 joints
Links:
- link link_0: mass None -> 0.2; geometry collision mesh filename=collision-body.obj scale=1.0 1.0 1.0; collision mesh filename=collision-handle.obj scale=1.0 1.0 1.0

File: models/StaplerFlat/103095/mobility.urdf (robot description, URDF)
Before this commit: robot partnet_376eb047b40ef4f6a480e3d8fdbd4a92, 4 links, 3 joints
Links:
- link link_0: mass None -> 0.2
- link link_1: mass None -> 0.2
- link link_2: mass None -> 0.2
Joints:
- joint joint_0: type revolute -> fixed
- joint joint_1: type revolute -> fixed
