Commit message: pack eyeglasses

File: models/Eyeglasses/101284/mobility.urdf (robot description, URDF)
Before this commit: robot partnet_1065a548dee0058d89cf6a343602477f, 4 links, 3 joints
Links:
- link link_0: mass None -> 0.2
- link link_1: mass None -> 0.2
- link link_2: mass None -> 0.2
Joints:
- joint joint_0: type revolute -> fixed
- joint joint_1: type revolute -> fixed
