Commit message: pack bottles

File: models/Bottle/3520/mobility.urdf (robot description, URDF)
Before this commit: robot partnet_2722bec1947151b86e22e2d2f64c8cef, 4 links, 3 joints
Links:
- link link_0: mass None -> 0.2
- link link_1: mass None -> 0.2
Joints:
- joint joint_0: type continuous -> fixed
- joint joint_2: type prismatic -> fixed

File: models/BottleOpened/3517/mobility.urdf (robot description, URDF)
Before this commit: robot partnet_917fd3e68de79bf69ece21a0b0786a69, 4 links, 3 joints
Links:
- removed link link_0
- removed link link_0_helper
- link link_1: mass None -> 1
Joints:
- removed joint joint_0
- removed joint joint_2

File: models/BottleOpened/3571/mobility.urdf (robot description, URDF)
Before this commit: robot partnet_1cf98e5b6fff5471c8724d5673a063a6, 4 links, 3 joints
Links:
- removed link link_0
- removed link link_0_helper
- link link_1: mass None -> 2
Joints:
- removed joint joint_0
- removed joint joint_2

File: models/Camera/101352/mobility.urdf (robot description, URDF)
Before this commit: robot partnet_1967344f80da29618d342172201b8d8c, 20 links, 19 joints
Links:
- link link_18: mass None -> 0.2
Joints:
- joint joint_0: type prismatic -> fixed
- joint joint_1: type prismatic -> fixed
- joint joint_10: type prismatic -> fixed
- joint joint_11: type prismatic -> fixed
- joint joint_12: type prismatic -> fixed
- joint joint_13: type prismatic -> fixed
- joint joint_14: type prismatic -> fixed
- joint joint_15: type prismatic -> fixed
- joint joint_16: type prismatic -> fixed
- joint joint_17: type prismatic -> fixed
- joint joint_2: type prismatic -> fixed
- joint joint_3: type prismatic -> fixed
- joint joint_4: type prismatic -> fixed
- joint joint_5: type prismatic -> fixed
- joint joint_6: type prismatic -> fixed
- joint joint_7: type continuous -> fixed
- joint joint_8: type prismatic -> fixed

File: models/Pliers/100144/mobility.urdf (robot description, URDF)
Before this commit: robot partnet_2f4b18402dee61003f7c6295b60afd1b, 3 links, 2 joints
Links:
- link link_0: mass None -> 0.2
- link link_1: mass None -> 0.2
Joints:
- joint joint_0: type revolute -> fixed

File: models/Scissors/10495/mobility.urdf (robot description, URDF)
Before this commit: robot partnet_3bba19a52cbe211cb458c00230942e4e, 3 links, 2 joints
Links:
- link link_0: mass None -> 0.2
- link link_1: mass None -> 0.2
Joints:
- joint joint_0: type revolute -> fixed
