Commit message: boc

File: models/BottleOpened/3571/mobility.urdf (robot description, URDF)
Before this commit: robot partnet_1cf98e5b6fff5471c8724d5673a063a6, 2 links, 1 joints
Links:
- link link_1: mass 2 -> 0.2

File: models/BottleOpened/3574/mobility.urdf (robot description, URDF)
Before this commit: robot partnet_1d4093ad2dfad9df24be2e4f911ee4af, 4 links, 3 joints
Links:
- removed link link_0
- removed link link_0_helper
- link link_1: mass None -> 0.2; geometry collision mesh filename=textured_objs/new-0.obj; collision mesh filename=textured_objs/new-1.obj
Joints:
- removed joint joint_0
- removed joint joint_2

File: models/BottleOpened/3593/mobility.urdf (robot description, URDF)
Before this commit: robot partnet_20c5dff3b09282035b76194468418a0e, 3 links, 2 joints
Links:
- removed link link_1
- link link_0: mass None -> 0.2
Joints:
- removed joint joint_1
