Commit message: box breakdown

File: models/Box/100426/mobility.urdf (robot description, URDF)
Before this commit: robot partnet_3e18df9aea04c8cdbc7fb81194b2b6a8, 4 links, 3 joints
Links:
- link link_2: geometry collision mesh filename=textured_objs/original-1.obj; collision mesh filename=textured_objs/original-5+x.obj
